Commit message: Fix gripper code not working when only 1 gripper move

File: urdf/baxter.urdf (robot description, URDF)
Before this commit: robot baxter, 57 links, 56 joints
Links:
- added link right_gripper_cube_offset, mass 0.0001
- link head: geometry collision sphere radius=0.001; visual mesh filename=/home/ubb/Documents/Baxter_isaac/ROS2/install/baxter_descri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
- link l_gripper_l_finger: geometry collision box size=0.01 0.0135 0.1127; collision box size=0.01 0.05 0.017
- link l_gripper_l_finger_tip: geometry collision box size=0.042 0.0065 0.037; visual mesh filename=/home/ubb/Documents/Baxter_isaac/ROS1/src/baxter_common/ret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
- link l_gripper_r_finger: geometry collision box size=0.01 0.0135 0.1127; collision box size=0.01 0.05 0.017
- link l_gripper_r_finger_tip: geometry collision box size=0.042 0.0065 0.037; visual mesh filename=/home/ubb/Documents/Baxter_isaac/ROS1/src/baxter_common/ret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
- link left_gripper_base: geometry collision cylinder length=0.1 radius=0.029; visual mesh filename=/home/ubb/Documents/Baxter_isaac/ROS2/install/rethink_ee_de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
- link left_lower_elbow: geometry collision cylinder length=0.10 radius=0.06; visual mesh filename=/home/ubb/Documents/Baxter_isaac/ROS2/install/baxter_descri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
- link left_lower_forearm: geometry collision cylinder length=0.10 radius=0.06; visual mesh filename=/home/ubb/Documents/Baxter_isaac/ROS2/install/baxter_descri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
- link left_lower_shoulder: geometry collision cylinder length=0.12 radius=0.06; visual mesh filename=/home/ubb/Documents/Baxter_isaac/ROS2/install/baxter_descri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
- link left_upper_elbow: geometry collision cylinder length=0.107 radius=0.06; visual mesh filename=/home/ubb/Documents/Baxter_isaac/ROS2/install/baxter_descri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
- link left_upper_forearm: geometry collision cylinder length=0.088 radius=0.06; visual mesh filename=/home/ubb/Documents/Baxter_isaac/ROS2/install/baxter_descri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
- link left_upper_shoulder: geometry collision cylinder length=0.2722 radius=0.06; visual mesh filename=/home/ubb/Documents/Baxter_isaac/ROS2/install/baxter_descri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
- link left_wrist: geometry collision cylinder length=0.165 radius=0.06; visual mesh filename=/home/ubb/Documents/Baxter_isaac/ROS2/install/baxter_descri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
- link pedestal: geometry collision mesh filename=/home/ubb/Documents/Baxter_isaac/ROS2/install/baxter_descri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; visual mesh filename=/home/ubb/Documents/Baxter_isaac/ROS2/install/baxter_descri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
- link r_gripper_l_finger: geometry collision box size=0.01 0.0135 0.1127; collision box size=0.01 0.05 0.017
- link r_gripper_l_finger_tip: geometry collision cylinder length=0.037 radius=0.008; visual mesh filename=/home/ubb/Documents/Baxter_isaac/ROS1/src/baxter_common/ret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
- link r_gripper_r_finger: geometry collision box size=0.01 0.0135 0.1127; collision box size=0.01 0.05 0.017
- link r_gripper_r_finger_tip: geometry collision cylinder length=0.037 radius=0.008; visual mesh filename=/home/ubb/Documents/Baxter_isaac/ROS1/src/baxter_common/ret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
- link right_gripper_base: geometry collision cylinder length=0.1 radius=0.029; visual mesh filename=/home/ubb/Documents/Baxter_isaac/ROS2/install/rethink_ee_de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
- link right_lower_elbow: geometry collision cylinder length=0.10 radius=0.06; visual mesh filename=/home/ubb/Documents/Baxter_isaac/ROS2/install/baxter_descri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
- link right_lower_forearm: geometry collision cylinder length=0.10 radius=0.06; visual mesh filename=/home/ubb/Documents/Baxter_isaac/ROS2/install/baxter_descri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
- link right_lower_shoulder: geometry collision cylinder length=0.12 radius=0.06; visual mesh filename=/home/ubb/Documents/Baxter_isaac/ROS2/install/baxter_descri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
- link right_upper_elbow: geometry collision cylinder length=0.107 radius=0.06; visual mesh filename=/home/ubb/Documents/Baxter_isaac/ROS2/install/baxter_descri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
- link right_upper_forearm: geometry collision cylinder length=0.088 radius=0.06; visual mesh filename=/home/ubb/Documents/Baxter_isaac/ROS2/install/baxter_descri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
- link right_upper_shoulder: geometry collision cylinder length=0.2722 radius=0.06; visual mesh filename=/home/ubb/Documents/Baxter_isaac/ROS2/install/baxter_descri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
- link right_wrist: geometry collision cylinder length=0.165 radius=0.06; visual mesh filename=/home/ubb/Documents/Baxter_isaac/ROS2/install/baxter_descri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
- link screen: geometry collision sphere radius=0.001; visual mesh filename=/home/ubb/Documents/Baxter_isaac/ROS2/install/baxter_descri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
- link torso: geometry collision mesh filename=/home/ubb/Documents/Baxter_isaac/ROS2/install/baxter_descri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; visual mesh filename=/home/ubb/Documents/Baxter_isaac/ROS2/install/baxter_descri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
Joints:
- added joint right_endpoint_offset: type fixed, parent right_gripper_base, child right_gripper_cube_offset, origin xyz=0 0 0.11269999999999998 rpy=0 0 0

Commit message: Update to Isaac 2022.2

File: urdf/baxter.urdf (robot description, URDF)
Before this commit: robot baxter, 58 links, 57 joints
Links:
- link r_gripper_l_finger_tip: geometry collision box size=0.042 0.0065 0.037; visual mesh filename=/home/ubb/Documents/Baxter_isaac/ROS1/src/baxter_common/ret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
- link r_gripper_r_finger_tip: geometry collision box size=0.042 0.0065 0.037; visual mesh filename=/home/ubb/Documents/Baxter_isaac/ROS1/src/baxter_common/ret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

Commit message: Fixes

File: urdf/baxter.urdf (robot description, URDF)
Before this commit: robot baxter, 58 links, 57 joints
Links:
- link head: geometry collision sphere radius=0.001; visual mesh filename=./baxter_description/meshes/head/H0.STL
- link l_gripper_l_finger: geometry collision box size=0.01 0.0135 0.1127; collision box size=0.01 0.05 0.017
- link l_gripper_l_finger_tip: geometry collision box size=0.042 0.0065 0.037; visual mesh filename=/rethink_ee_description/meshes/electric_gripper/fingers/pad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
- link l_gripper_r_finger: geometry collision box size=0.01 0.0135 0.1127; collision box size=0.01 0.05 0.017
- link l_gripper_r_finger_tip: geometry collision box size=0.042 0.0065 0.037; visual mesh filename=/rethink_ee_description/meshes/electric_gripper/fingers/pad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
- link left_gripper_base: geometry collision cylinder length=0.1 radius=0.029; visual mesh filename=/rethink_ee_description/share//rethink_ee_description/meshe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
- link left_lower_elbow: geometry collision cylinder length=0.10 radius=0.06; visual mesh filename=./baxter_description/meshes/lower_elbow/E1.DAE
- link left_lower_forearm: geometry collision cylinder length=0.10 radius=0.06; visual mesh filename=./baxter_description/meshes/lower_forearm/W1.DAE
- link left_lower_shoulder: geometry collision cylinder length=0.12 radius=0.06; visual mesh filename=./baxter_description/meshes/lower_shoulder/S1.DAE
- link left_upper_elbow: geometry collision cylinder length=0.107 radius=0.06; visual mesh filename=./baxter_description/meshes/upper_elbow/E0.DAE
- link left_upper_forearm: geometry collision cylinder length=0.088 radius=0.06; visual mesh filename=./baxter_description/meshes/upper_forearm/W0.DAE
- link left_upper_shoulder: geometry collision cylinder length=0.2722 radius=0.06; visual mesh filename=./baxter_description/meshes/upper_shoulder/S0.DAE
- link left_wrist: geometry collision cylinder length=0.165 radius=0.06; visual mesh filename=./baxter_description/meshes/wrist/W2.DAE
- link pedestal: geometry collision mesh filename=./baxter_description/meshes/base/pedestal_link_collision.DAE; visual mesh filename=./baxter_description/meshes/base/PEDESTAL.DAE
- link r_gripper_l_finger: geometry collision box size=0.01 0.0135 0.1127; collision box size=0.01 0.05 0.017
- link r_gripper_l_finger_tip: geometry collision box size=0.042 0.0065 0.037; visual mesh filename=/rethink_ee_description/meshes/electric_gripper/fingers/pad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
- link r_gripper_r_finger: geometry collision box size=0.01 0.0135 0.1127; collision box size=0.01 0.05 0.017
- link r_gripper_r_finger_tip: geometry collision box size=0.042 0.0065 0.037; visual mesh filename=/rethink_ee_description/meshes/electric_gripper/fingers/pad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
- link right_gripper_base: geometry collision cylinder length=0.1 radius=0.029; visual mesh filename=/rethink_ee_description/share//rethink_ee_description/meshe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
- link right_lower_elbow: geometry collision cylinder length=0.10 radius=0.06; visual mesh filename=./baxter_description/meshes/lower_elbow/E1.DAE
- link right_lower_forearm: geometry collision cylinder length=0.10 radius=0.06; visual mesh filename=./baxter_description/meshes/lower_forearm/W1.DAE
- link right_lower_shoulder: geometry collision cylinder length=0.12 radius=0.06; visual mesh filename=./baxter_description/meshes/lower_shoulder/S1.DAE
- link right_upper_elbow: geometry collision cylinder length=0.107 radius=0.06; visual mesh filename=./baxter_description/meshes/upper_elbow/E0.DAE
- link right_upper_forearm: geometry collision cylinder length=0.088 radius=0.06; visual mesh filename=./baxter_description/meshes/upper_forearm/W0.DAE
- link right_upper_shoulder: geometry collision cylinder length=0.2722 radius=0.06; visual mesh filename=./baxter_description/meshes/upper_shoulder/S0.DAE
- link right_wrist: geometry collision cylinder length=0.165 radius=0.06; visual mesh filename=./baxter_description/meshes/wrist/W2.DAE
- link screen: geometry collision sphere radius=0.001; visual mesh filename=./baxter_description/meshes/head/H1.DAE
- link torso: geometry collision mesh filename=./baxter_description/meshes/torso/base_link_collision.DAE; visual mesh filename=./baxter_description/meshes/torso/base_link.DAE

Commit message: Removed hardcoded path

File: urdf/baxter.urdf (robot description, URDF)
Before this commit: robot baxter, 58 links, 57 joints
Links:
- link head: geometry collision sphere radius=0.001; visual mesh filename=package://baxter_description/meshes/head/H0.DAE
- link l_gripper_l_finger: geometry collision box size=0.01 0.0135 0.1127; collision box size=0.01 0.05 0.017
- link l_gripper_l_finger_tip: geometry collision box size=0.042 0.0065 0.037; visual mesh filename=package://rethink_ee_description/meshes/electric_gripper/fi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
- link l_gripper_r_finger: geometry collision box size=0.01 0.0135 0.1127; collision box size=0.01 0.05 0.017
- link l_gripper_r_finger_tip: geometry collision box size=0.042 0.0065 0.037; visual mesh filename=package://rethink_ee_description/meshes/electric_gripper/fi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
- link left_gripper_base: geometry collision cylinder length=0.1 radius=0.029; visual mesh filename=package://rethink_ee_description/meshes/electric_gripper/el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
- link left_lower_elbow: geometry collision cylinder length=0.10 radius=0.06; visual mesh filename=package://baxter_description/meshes/lower_elbow/E1.DAE
- link left_lower_forearm: geometry collision cylinder length=0.10 radius=0.06; visual mesh filename=package://baxter_description/meshes/lower_forearm/W1.DAE
- link left_lower_shoulder: geometry collision cylinder length=0.12 radius=0.06; visual mesh filename=package://baxter_description/meshes/lower_shoulder/S1.DAE
- link left_upper_elbow: geometry collision cylinder length=0.107 radius=0.06; visual mesh filename=package://baxter_description/meshes/upper_elbow/E0.DAE
- link left_upper_forearm: geometry collision cylinder length=0.088 radius=0.06; visual mesh filename=package://baxter_description/meshes/upper_forearm/W0.DAE
- link left_upper_shoulder: geometry collision cylinder length=0.2722 radius=0.06; visual mesh filename=package://baxter_description/meshes/upper_shoulder/S0.DAE
- link left_wrist: geometry collision cylinder length=0.165 radius=0.06; visual mesh filename=package://baxter_description/meshes/wrist/W2.DAE
- link pedestal: geometry collision mesh filename=package://baxter_description/meshes/base/pedestal_link_coll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; visual mesh filename=package://baxter_description/meshes/base/PEDESTAL.DAE
- link r_gripper_l_finger: geometry collision box size=0.01 0.0135 0.1127; collision box size=0.01 0.05 0.017
- link r_gripper_l_finger_tip: geometry collision box size=0.042 0.0065 0.037; visual mesh filename=package://rethink_ee_description/meshes/electric_gripper/fi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
- link r_gripper_r_finger: geometry collision box size=0.01 0.0135 0.1127; collision box size=0.01 0.05 0.017
- link r_gripper_r_finger_tip: geometry collision box size=0.042 0.0065 0.037; visual mesh filename=package://rethink_ee_description/meshes/electric_gripper/fi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
- link right_gripper_base: geometry collision cylinder length=0.1 radius=0.029; visual mesh filename=package://rethink_ee_description/meshes/electric_gripper/el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
- link right_lower_elbow: geometry collision cylinder length=0.10 radius=0.06; visual mesh filename=package://baxter_description/meshes/lower_elbow/E1.DAE
- link right_lower_forearm: geometry collision cylinder length=0.10 radius=0.06; visual mesh filename=package://baxter_description/meshes/lower_forearm/W1.DAE
- link right_lower_shoulder: geometry collision cylinder length=0.12 radius=0.06; visual mesh filename=package://baxter_description/meshes/lower_shoulder/S1.DAE
- link right_upper_elbow: geometry collision cylinder length=0.107 radius=0.06; visual mesh filename=package://baxter_description/meshes/upper_elbow/E0.DAE
- link right_upper_forearm: geometry collision cylinder length=0.088 radius=0.06; visual mesh filename=package://baxter_description/meshes/upper_forearm/W0.DAE
- link right_upper_shoulder: geometry collision cylinder length=0.2722 radius=0.06; visual mesh filename=package://baxter_description/meshes/upper_shoulder/S0.DAE
- link right_wrist: geometry collision cylinder length=0.165 radius=0.06; visual mesh filename=package://baxter_description/meshes/wrist/W2.DAE
- link screen: geometry collision sphere radius=0.001; visual mesh filename=package://baxter_description/meshes/head/H1.DAE
- link torso: geometry collision mesh filename=package://baxter_description/meshes/torso/base_link_collisi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; visual mesh filename=package://baxter_description/meshes/torso/base_link.DAE
